File: switch-matrix.sch (KiCad schematic (older format))
At the start: 0 parts

Commit message: Started work on switch matrix.
Parts:
- added C? (x4): CYA, ~, symbol C
- added D? (x4): ZENERSMALL, ~, symbol ZENERSMALL
- added D? (x16): DIODE, ~, symbol DIODE
- added Q? (x4): NPN, ~, symbol NPN
- added RP? (x5): R_PACK4, ~, symbol R_PACK4
- added U? (x4): 74HC14, ~, symbol 74HC14
Connections:
- net labels added: +12V, +3.3V, COL0_POWERED, COL1_POWERED, COL2_POWERED, COL3_POWERED, GND, ROW0_MATRIX, ROW1_MATRIX, ROW2_MATRIX, ROW3_MATRIX
- wire segments 0 -> 135

Commit message: Added library for custom parts Switch matrix and solenoid driver mostly done
Parts:
- removed D? (x16): DIODE, ~, symbol DIODE
- added C1: 100n, ~, symbol C
- added D10, D11, D12, D5, D6, D7, D8, D9: BAT54C, ~, symbol DOUBLE_SCH_KCOM
- added P1, P2, P3, P4: CONN_8, symbol CONN_8
- gave numbers to parts that had none: 18
Connections:
- wire segments 135 -> 175

Commit message: Updating switch matrix to use pullups on row inputs rather than pulldowns, so that it will actually work
Connections:
- wire segments 175 -> 183
Other:
- moved on the sheet: RP2, RP4
Changed lines of the file:
@@
-EESchema Schematic File Version 2  date 4/10/2013 12:44:15 AM
+EESchema Schematic File Version 2  date 4/10/2013 12:52:04 AM
 LIBS:power
 LIBS:device
@@
 L R_PACK4 RP2
 U 1 1 51644B2D
-P 6250 1900
-F 0 "RP2" H 6250 2350 40  0000 C CNN
-F 1 "R_PACK4" H 6250 1850 40  0000 C CNN
-F 2 "~" H 6250 1900 60  0000 C CNN
-F 3 "~" H 6250 1900 60  0000 C CNN
-	1    6250 1900
+P 6550 1900
+F 0 "RP2" H 6550 2350 40  0000 C CNN
+F 1 "R_PACK4" H 6550 1850 40  0000 C CNN
+F 2 "~" H 6550 1900 60  0000 C CNN
+F 3 "~" H 6550 1900 60  0000 C CNN
+	1    6550 1900
 	1    0    0    -1
 $EndComp
@@
 L R_PACK4 RP4
 U 1 1 51644B3C
-P 6250 2800
-F 0 "RP4" H 6250 3250 40  0000 C CNN
-F 1 "R_PACK4" H 6250 2750 40  0000 C CNN
-F 2 "~" H 6250 2800 60  0000 C CNN
-F 3 "~" H 6250 2800 60  0000 C CNN
-	1    6250 2800
+P 6550 1250
+F 0 "RP4" H 6550 1700 40  0000 C CNN
+F 1 "R_PACK4" H 6550 1200 40  0000 C CNN
+F 2 "~" H 6550 1250 60  0000 C CNN
+F 3 "~" H 6550 1250 60  0000 C CNN
+	1    6550 1250
 	1    0    0    -1
 $EndComp
@@
 L +12V #PWR1
 U 1 1 51644F71
-P 1700 850
-F 0 "#PWR1" H 1700 800 20  0001 C CNN
-F 1 "+12V" H 1700 950 30  0000 C CNN
-F 2 "" H 1700 850 60  0000 C CNN
-F 3 "" H 1700 850 60  0000 C CNN
-	1    1700 850
+P 1700 900
+F 0 "#PWR1" H 1700 850 20  0001 C CNN
+F 1 "+12V" H 1700 1000 30  0000 C CNN
+F 2 "" H 1700 900 60  0000 C CNN
+F 3 "" H 1700 900 60  0000 C CNN
+	1    1700 900
 	1    0    0    -1
 $EndComp
@@
 	1700 1300 1800 1300
 Wire Wire Line
-	1700 850  1700 1300
+	1700 900  1700 1300
 Wire Wire Line
 	1800 1200 1700 1200
@@
 Connection ~ 1700 1000
 Wire Wire Line
-	6450 2450 8550 2450
-Wire Wire Line
 	6650 2450 6650 2950
 Wire Wire Line
 	6850 1850 6850 2850
-Connection ~ 6650 2450
-Wire Wire Line
-	6450 2550 8650 2550
 Wire Wire Line
 	7150 2550 7150 2950
 Wire Wire Line
 	7350 1750 7350 2850
-Connection ~ 7150 2550
-Wire Wire Line
-	6450 2650 8650 2650
 Wire Wire Line
 	7650 2650 7650 2950
 Wire Wire Line
 	7850 1650 7850 2850
-Connection ~ 7650 2650
-Wire Wire Line
-	6450 2750 8550 2750
 Wire Wire Line
 	8150 2750 8150 2950
 Wire Wire Line
 	8350 1550 8350 2850
-Connection ~ 8150 2750
 Wire Wire Line
 	8350 3350 8350 3250
 Wire Wire Line
-	5950 3350 8350 3350
-Wire Wire Line
-	6650 3350 6650 3150
+	6650 3150 6650 3450
 Wire Wire Line
 	6850 3250 6850 3350
 Connection ~ 6850 3350
 Wire Wire Line
-	7150 3150 7150 3350
+	7150 3350 7150 3150
 Connection ~ 7150 3350
 Wire Wire Line
-	7350 3250 7350 3350
+	7350 3350 7350 3250
 Connection ~ 7350 3350
 Wire Wire Line
-	7650 3150 7650 3350
+	7650 3350 7650 3150
 Connection ~ 7650 3350
 Wire Wire Line
-	7850 3250 7850 3350
+	7850 3350 7850 3250
 Connection ~ 7850 3350
 Wire Wire Line
-	8150 3150 8150 3350
+	8150 3350 8150 3150
 Connection ~ 8150 3350
 Wire Wire Line
-	6450 1850 6850 1850
+	6750 1850 6850 1850
 Connection ~ 6850 2450
 Wire Wire Line
-	6450 1750 7350 1750
+	6750 1750 7350 1750
 Connection ~ 7350 2550
 Wire Wire Line
-	6450 1650 7850 1650
+	6750 1650 7850 1650
 Connection ~ 7850 2650
 Wire Wire Line
-	6450 1550 8350 1550
+	6750 1550 8350 1550
 Connection ~ 8350 2750
-Wire Wire Line
-	5950 2450 5950 3450
-Wire Wire Line
-	5950 2450 6050 2450
 Connection ~ 6650 3350
-Wire Wire Line
-	6050 2550 5950 2550
-Connection ~ 5950 2550
-Wire Wire Line
-	6050 2650 5950 2650
-Connection ~ 5950 2650
-Wire Wire Line
-	6050 2750 5950 2750
-Connection ~ 5950 2750
 $Comp
 L GND #PWR8
 U 1 1 51645A06
-P 5950 3450
-F 0 "#PWR8" H 5950 3450 30  0001 C CNN
-F 1 "GND" H 5950 3380 30  0001 C CNN
-F 2 "" H 5950 3450 60  0000 C CNN
-F 3 "" H 5950 3450 60  0000 C CNN
-	1    5950 3450
-	1    0    0    -1
-$EndComp
-Connection ~ 5950 3350
+P 6650 3450
+F 0 "#PWR8" H 6650 3450 30  0001 C CNN
+F 1 "GND" H 6650 3380 30  0001 C CNN
+F 2 "" H 6650 3450 60  0000 C CNN
+F 3 "" H 6650 3450 60  0000 C CNN
+	1    6650 3450
+	1    0    0    -1
+$EndComp
 Text Label 4850 1650 2    60   ~ 0
 COL0_POWERED
@@
 ROW3_MATRIX
 Wire Wire Line
-	5250 1850 6050 1850
-Wire Wire Line
-	6050 1750 5250 1750
-Wire Wire Line
-	5250 1650 6050 1650
-Wire Wire Line
-	6050 1550 5250 1550
+	5250 1850 6350 1850
+Wire Wire Line
+	5250 1750 6350 1750
+Wire Wire Line
+	5250 1650 6350 1650
+Wire Wire Line
+	5250 1550 6350 1550
 Wire Wire Line
 	10050 2050 9850 2050
@@
 Wire Wire Line
 	9850 1350 9850 1300
+Wire Wire Line
+	6650 3350 8350 3350
+Wire Wire Line
+	8550 2750 8150 2750
+Wire Wire Line
+	7650 2650 8650 2650
+Wire Wire Line
+	8650 2550 7150 2550
+Wire Wire Line
+	8550 2450 6650 2450
+Wire Wire Line
+	6250 1200 6350 1200
+Wire Wire Line
+	6250 1200 6250 1850
+Connection ~ 6250 1850
+Wire Wire Line
+	6350 1100 6150 1100
+Wire Wire Line
+	6150 1100 6150 1750
+Connection ~ 6150 1750
+Wire Wire Line
+	6350 1000 6050 1000
+Wire Wire Line
+	6050 1000 6050 1650
+Connection ~ 6050 1650
+Wire Wire Line
+	6350 900  5950 900
+Wire Wire Line
+	5950 900  5950 1550
+Connection ~ 5950 1550
+$Comp
+L +12V #PWR?
+U 1 1 516506D2
+P 6850 800
+F 0 "#PWR?" H 6850 750 20  0001 C CNN
+F 1 "+12V" H 6850 900 30  0000 C CNN
+F 2 "" H 6850 800 60  0000 C CNN
+F 3 "" H 6850 800 60  0000 C CNN
+	1    6850 800
+	1    0    0    -1
+$EndComp
+Wire Wire Line
+	6750 1200 6850 1200
+Wire Wire Line
+	6850 1200 6850 800
+Wire Wire Line
+	6750 900  6850 900
+Connection ~ 6850 900
+Wire Wire Line
+	6750 1000 6850 1000
+Connection ~ 6850 1000
+Wire Wire Line
+	6750 1100 6850 1100
+Connection ~ 6850 1100
 $EndSCHEMATC

Commit message: Fixed switch matrix to match Mike's sketches Added lamp matrix
Connections:
- wire segments 183 -> 175
Other:
- moved on the sheet: D5, D7, P1, RP4
