File: switch-matrix.sch (KiCad schematic (older format))
At the start: 31 parts, among them P1 CONN_8, P2 CONN_8, P3 CONN_8, P4 CONN_8, Q1 NPN, Q2 NPN, Q3 NPN, Q4 NPN, U1 74HC14

Commit message: added dip switch library and modifed current sense's to add capsstarted the main controller page
Parts:
- P1: value CONN_8 -> SW_0
- P2: value CONN_8 -> SW_1
- P3: value CONN_8 -> SW_2
- P4: value CONN_8 -> SW_3
Connections:
- net labels added: 12V_IN, SW_PWR
- net labels removed: +12V
- wire segments 175 -> 176
Changed lines of the file:
@@
-EESchema Schematic File Version 2  date 4/16/2013 2:34:18 AM
+EESchema Schematic File Version 2  date 4/16/2013 9:07:53 PM
 LIBS:power
 LIBS:device
@@
 LIBS:CurrentSense
 LIBS:pinball-power
+LIBS:dips-s
 LIBS:base-module-cache
 EELAYER 27 0
@@
 Sheet 2 10
 Title ""
-Date "16 apr 2013"
+Date "17 apr 2013"
 Rev ""
 Comp ""
@@
 	1    0    0    -1
 $EndComp
-$Comp
-L +12V #PWR1
-U 1 1 51644F71
-P 1700 900
-F 0 "#PWR1" H 1700 850 20  0001 C CNN
-F 1 "+12V" H 1700 1000 30  0000 C CNN
-F 2 "" H 1700 900 60  0000 C CNN
-F 3 "" H 1700 900 60  0000 C CNN
-	1    1700 900
-	1    0    0    -1
-$EndComp
 Wire Wire Line
 	1000 1950 1800 1950
@@
 	1700 1300 1800 1300
 Wire Wire Line
-	1700 900  1700 1300
+	1700 950  1700 1300
 Wire Wire Line
 	1800 1200 1700 1200
@@
 	6650 3150 6650 3450
 Wire Wire Line
-	6850 3250 6850 3350
+	6850 3350 6850 3250
 Connection ~ 6850 3350
 Wire Wire Line
@@
 P 2900 4450
 F 0 "P1" V 2850 4450 60  0000 C CNN
-F 1 "CONN_8" V 2950 4450 60  0000 C CNN
+F 1 "SW_0" V 2950 4450 60  0000 C CNN
 F 2 "" H 2900 4450 60  0000 C CNN
 F 3 "" H 2900 4450 60  0000 C CNN
@@
 Connection ~ 7650 2650
 Wire Wire Line
-	5950 3350 5950 2450
+	5950 2450 5950 3350
 Wire Wire Line
 	5950 2450 6050 2450
@@
 P 5500 4450
 F 0 "P2" V 5450 4450 60  0000 C CNN
-F 1 "CONN_8" V 5550 4450 60  0000 C CNN
+F 1 "SW_1" V 5550 4450 60  0000 C CNN
 F 2 "" H 5500 4450 60  0000 C CNN
 F 3 "" H 5500 4450 60  0000 C CNN
@@
 P 2900 5800
 F 0 "P3" V 2850 5800 60  0000 C CNN
-F 1 "CONN_8" V 2950 5800 60  0000 C CNN
+F 1 "SW_2" V 2950 5800 60  0000 C CNN
 F 2 "" H 2900 5800 60  0000 C CNN
 F 3 "" H 2900 5800 60  0000 C CNN
@@
 P 5500 5800
 F 0 "P4" V 5450 5800 60  0000 C CNN
-F 1 "CONN_8" V 5550 5800 60  0000 C CNN
+F 1 "SW_3" V 5550 5800 60  0000 C CNN
 F 2 "" H 5500 5800 60  0000 C CNN
 F 3 "" H 5500 5800 60  0000 C CNN
@@
 Text Label 4700 6450 2    60   ~ 0
 ROW3_MATRIX
+Text HLabel 1050 950  0    60   Input ~ 0
+12V_IN
+Wire Wire Line
+	1050 950  1700 950
+Text Label 1450 950  0    60   ~ 0
+SW_PWR
 $EndSCHEMATC
