File: solenoid-driver.sch (KiCad schematic (older format))
At the start: 60 parts, among them Q10 NPN, Q11 DUAL_MOSFET_N, Q12 NPN, Q13 NPN, Q14 DUAL_MOSFET_N, Q15 NPN, Q16 NPN, Q5 DUAL_MOSFET_N, Q6 NPN, Q7 NPN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

Commit message: added the other two current sense outputs and modified the power circut, i cant seem to add the 9th pad, the bottom thermal pad????
Connections:
- net labels added: SOL_PWR, SOL_PWR_IN
- net labels removed: +48V, SOLENOID_CURRENT
- wire segments 280 -> 281
