File: 3V3CurrentSense.sch (KiCad schematic (older format))
At the start: 3 parts

Commit message: changed the controller adding some shift registers
Parts:
- gave numbers to parts that had none: 3
Changed lines of the file:
@@
-EESchema Schematic File Version 2  date 4/16/2013 9:07:53 PM
+EESchema Schematic File Version 2  date 4/17/2013 1:22:00 AM
 LIBS:power
 LIBS:device
@@
 LIBS:pinball-power
 LIBS:dips-s
+LIBS:Gajda_cmosieee
+LIBS:Gajda_ttlieee
 LIBS:base-module-cache
 EELAYER 27 0
@@
 SENSE_OUT
 $Comp
-L TS1102 U?
+L TS1102 U6
 U 1 1 516D5D2F
 P 5400 4100
-F 0 "U?" H 5600 4550 60  0000 C CNN
+AR Path="/516D5B3C/516D5D2F" Ref="U6"  Part="1"
+AR Path="/516D6DB7/516D5D2F" Ref="U7"  Part="1"
+F 0 "U7" H 5600 4550 60  0000 C CNN
 F 1 "TS1102" H 5500 4450 60  0000 C CNN
 F 2 "" H 5200 4100 60  0000 C CNN
@@
 $EndComp
 $Comp
-L R R?
+L R R48
 U 1 1 516D5D3E
 P 2750 2850
-F 0 "R?" V 2830 2850 40  0000 C CNN
+AR Path="/516D5B3C/516D5D3E" Ref="R48"  Part="1"
+AR Path="/516D6DB7/516D5D3E" Ref="R49"  Part="1"
+F 0 "R49" V 2830 2850 40  0000 C CNN
 F 1 "R" V 2757 2851 40  0000 C CNN
 F 2 "~" V 2680 2850 30  0000 C CNN
@@
 	3000 2850 3750 2850
 $Comp
-L GND #PWR?
+L GND #PWR41
 U 1 1 516D5D66
 P 5500 4750
-F 0 "#PWR?" H 5500 4750 30  0001 C CNN
+AR Path="/516D5B3C/516D5D66" Ref="#PWR41"  Part="1"
+AR Path="/516D6DB7/516D5D66" Ref="#PWR44"  Part="1"
+F 0 "#PWR44" H 5500 4750 30  0001 C CNN
 F 1 "GND" H 5500 4680 30  0001 C CNN
 F 2 "" H 5500 4750 60  0000 C CNN
@@
 $EndComp
 $Comp
-L GND #PWR?
+L GND #PWR42
 U 1 1 516D5D73
 P 5600 4750
-F 0 "#PWR?" H 5600 4750 30  0001 C CNN
+AR Path="/516D5B3C/516D5D73" Ref="#PWR42"  Part="1"
+AR Path="/516D6DB7/516D5D73" Ref="#PWR45"  Part="1"
+F 0 "#PWR45" H 5600 4750 30  0001 C CNN
 F 1 "GND" H 5600 4680 30  0001 C CNN
 F 2 "" H 5600 4750 60  0000 C CNN
@@
 	5500 4600 5500 4750
 $Comp
-L C C?
+L C C16
 U 1 1 516D5FD3
 P 6250 4400
-F 0 "C?" H 6250 4500 40  0000 L CNN
+AR Path="/516D5B3C/516D5FD3" Ref="C16"  Part="1"
+AR Path="/516D6DB7/516D5FD3" Ref="C17"  Part="1"
+F 0 "C17" H 6250 4500 40  0000 L CNN
 F 1 "0.047uF" H 6256 4315 40  0000 L CNN
 F 2 "~" H 6288 4250 30  0000 C CNN
@@
 Connection ~ 6250 4100
 $Comp
-L GND #PWR?
+L GND #PWR43
 U 1 1 516D5FF7
 P 6250 4750
-F 0 "#PWR?" H 6250 4750 30  0001 C CNN
+AR Path="/516D5B3C/516D5FF7" Ref="#PWR43"  Part="1"
+AR Path="/516D6DB7/516D5FF7" Ref="#PWR46"  Part="1"
+F 0 "#PWR46" H 6250 4750 30  0001 C CNN
 F 1 "GND" H 6250 4680 30  0001 C CNN
 F 2 "" H 6250 4750 60  0000 C CNN
