File: 3V3CurrentSense_2.sch (KiCad schematic (older format))
At the start: 3 parts, among them U6 TS1102

Commit message: ran an ERC and touched up a couple small issues
Changed lines of the file:
@@
-EESchema Schematic File Version 2  date 4/18/2013 1:06:20 AM
+EESchema Schematic File Version 2  date 4/18/2013 1:12:38 AM
 LIBS:power
 LIBS:device
@@
 $Descr A4 11693 8268
 encoding utf-8
-Sheet 9 10
+Sheet 8 10
 Title ""
 Date "18 apr 2013"
@@
 AR Path="/516D5B3C/516D5D2F" Ref="U6"  Part="1"
 AR Path="/516D6DB7/516D5D2F" Ref="U7"  Part="1"
-F 0 "U7" H 5600 4550 60  0000 C CNN
+F 0 "U6" H 5600 4550 60  0000 C CNN
 F 1 "TS1102" H 5500 4450 60  0000 C CNN
 F 2 "" H 5200 4100 60  0000 C CNN
@@
 AR Path="/516D5B3C/516D5D3E" Ref="R52"  Part="1"
 AR Path="/516D6DB7/516D5D3E" Ref="R53"  Part="1"
-F 0 "R53" V 2830 2850 40  0000 C CNN
+F 0 "R52" V 2830 2850 40  0000 C CNN
 F 1 "R" V 2757 2851 40  0000 C CNN
 F 2 "~" V 2680 2850 30  0000 C CNN
@@
 AR Path="/516D5B3C/516D5FD3" Ref="C16"  Part="1"
 AR Path="/516D6DB7/516D5FD3" Ref="C17"  Part="1"
-F 0 "C17" H 6250 4500 40  0000 L CNN
+F 0 "C16" H 6250 4500 40  0000 L CNN
 F 1 "0.047uF" H 6256 4315 40  0000 L CNN
 F 2 "~" H 6288 4250 30  0000 C CNN
