File: CurrentSense.sch (KiCad schematic (older format))
At the start: 5 parts

Commit message: added dip switch library and modifed current sense's to add capsstarted the main controller page
Parts:
- added C? (x2): 100nF, ~, symbol C
Connections:
- net +5V: now also C?.1, C?.1
- net GND: now also C?.2, C?.2
Changed lines of the file:
@@
-EESchema Schematic File Version 2  date 4/16/2013 2:34:18 AM
+EESchema Schematic File Version 2  date 4/16/2013 9:07:53 PM
 LIBS:power
 LIBS:device
@@
 LIBS:CurrentSense
 LIBS:pinball-power
+LIBS:dips-s
 LIBS:base-module-cache
 EELAYER 27 0
@@
 Sheet 7 10
 Title ""
-Date "16 apr 2013"
+Date "17 apr 2013"
 Rev ""
 Comp ""
@@
 	7050 3750 7400 3750
 Connection ~ 7250 3750
+$Comp
+L C C?
+U 1 1 516E8E76
+P 4950 2500
+F 0 "C?" H 4950 2600 40  0000 L CNN
+F 1 "100nF" H 4956 2415 40  0000 L CNN
+F 2 "~" H 4988 2350 30  0000 C CNN
+F 3 "~" H 4950 2500 60  0000 C CNN
+	1    4950 2500
+	1    0    0    -1
+$EndComp
+$Comp
+L +5V #PWR?
+U 1 1 516E8E83
+P 4950 2250
+F 0 "#PWR?" H 4950 2340 20  0001 C CNN
+F 1 "+5V" H 4950 2340 30  0000 C CNN
+F 2 "" H 4950 2250 60  0000 C CNN
+F 3 "" H 4950 2250 60  0000 C CNN
+	1    4950 2250
+	1    0    0    -1
+$EndComp
+$Comp
+L GND #PWR?
+U 1 1 516E8E8F
+P 4950 2750
+F 0 "#PWR?" H 4950 2750 30  0001 C CNN
+F 1 "GND" H 4950 2680 30  0001 C CNN
+F 2 "" H 4950 2750 60  0000 C CNN
+F 3 "" H 4950 2750 60  0000 C CNN
+	1    4950 2750
+	1    0    0    -1
+$EndComp
+Wire Wire Line
+	4950 2300 4950 2250
+Wire Wire Line
+	4950 2700 4950 2750
+$Comp
+L C C?
+U 1 1 516E8ED2
+P 6350 2500
+F 0 "C?" H 6350 2600 40  0000 L CNN
+F 1 "100nF" H 6356 2415 40  0000 L CNN
+F 2 "~" H 6388 2350 30  0000 C CNN
+F 3 "~" H 6350 2500 60  0000 C CNN
+	1    6350 2500
+	1    0    0    -1
+$EndComp
+$Comp
+L +5V #PWR?
+U 1 1 516E8ED8
+P 6350 2250
+F 0 "#PWR?" H 6350 2340 20  0001 C CNN
+F 1 "+5V" H 6350 2340 30  0000 C CNN
+F 2 "" H 6350 2250 60  0000 C CNN
+F 3 "" H 6350 2250 60  0000 C CNN
+	1    6350 2250
+	1    0    0    -1
+$EndComp
+$Comp
+L GND #PWR?
+U 1 1 516E8EDE
+P 6350 2750
+F 0 "#PWR?" H 6350 2750 30  0001 C CNN
+F 1 "GND" H 6350 2680 30  0001 C CNN
+F 2 "" H 6350 2750 60  0000 C CNN
+F 3 "" H 6350 2750 60  0000 C CNN
+	1    6350 2750
+	1    0    0    -1
+$EndComp
+Wire Wire Line
+	6350 2300 6350 2250
+Wire Wire Line
+	6350 2700 6350 2750
 $EndSCHEMATC

Commit message: changed the controller adding some shift registers
Parts:
- gave numbers to parts that had none: 7
Changed lines of the file:
@@
-EESchema Schematic File Version 2  date 4/16/2013 9:07:53 PM
+EESchema Schematic File Version 2  date 4/17/2013 1:22:00 AM
 LIBS:power
 LIBS:device
@@
 LIBS:pinball-power
 LIBS:dips-s
+LIBS:Gajda_cmosieee
+LIBS:Gajda_ttlieee
 LIBS:base-module-cache
 EELAYER 27 0
@@
 $EndDescr
 $Comp
-L LMP8480_/_LMP8481 U?
+L LMP8480_/_LMP8481 U4
 U 1 1 516CAFE0
 P 4150 3600
-F 0 "U?" H 3150 4450 60  0000 C CNN
+F 0 "U4" H 3150 4450 60  0000 C CNN
 F 1 "LMP8480_/_LMP8481" H 3600 4350 60  0000 C CNN
 F 2 "~" H 3500 3600 60  0000 C CNN
@@
 $EndComp
 $Comp
-L R R?
+L R R45
 U 1 1 516CAFEF
 P 2450 2550
-F 0 "R?" V 2530 2550 40  0000 C CNN
+F 0 "R45" V 2530 2550 40  0000 C CNN
 F 1 "R" V 2457 2551 40  0000 C CNN
 F 2 "~" V 2380 2550 30  0000 C CNN
@@
 	2700 3350 2700 2550
 $Comp
-L +5V #PWR?
+L +5V #PWR31
 U 1 1 516CB005
 P 4150 2700
-F 0 "#PWR?" H 4150 2790 20  0001 C CNN
+F 0 "#PWR31" H 4150 2790 20  0001 C CNN
 F 1 "+5V" H 4150 2790 30  0000 C CNN
 F 2 "" H 4150 2700 60  0000 C CNN
@@
 	4150 2700 4150 2850
 $Comp
-L GND #PWR?
+L GND #PWR32
 U 1 1 516CB018
 P 4400 3050
-F 0 "#PWR?" H 4400 3050 30  0001 C CNN
+F 0 "#PWR32" H 4400 3050 30  0001 C CNN
 F 1 "GND" H 4400 2980 30  0001 C CNN
 F 2 "" H 4400 3050 60  0000 C CNN
@@
 	4300 2900 4300 3000
 $Comp
-L R R?
+L R R46
 U 1 1 516CB283
 P 7250 4150
-F 0 "R?" V 7330 4150 40  0000 C CNN
+F 0 "R46" V 7330 4150 40  0000 C CNN
 F 1 "680" V 7257 4151 40  0000 C CNN
 F 2 "~" V 7180 4150 30  0000 C CNN
@@
 $EndComp
 $Comp
-L R R?
+L R R47
 U 1 1 516CB291
 P 7250 4750
-F 0 "R?" V 7330 4750 40  0000 C CNN
+F 0 "R47" V 7330 4750 40  0000 C CNN
 F 1 "1K" V 7257 4751 40  0000 C CNN
 F 2 "~" V 7180 4750 30  0000 C CNN
@@
 SNS_OUT
 $Comp
-L GND #PWR?
+L GND #PWR39
 U 1 1 516CB2F2
 P 7250 5100
-F 0 "#PWR?" H 7250 5100 30  0001 C CNN
+F 0 "#PWR39" H 7250 5100 30  0001 C CNN
 F 1 "GND" H 7250 5030 30  0001 C CNN
 F 2 "" H 7250 5100 60  0000 C CNN
@@
 1K/(1K+680)*5=3 (2.976190476)
 $Comp
-L MCP6001 U?
+L MCP6001 U5
 U 1 1 516CC857
 P 6350 3750
-F 0 "U?" H 6050 4300 60  0000 C CNN
+F 0 "U5" H 6050 4300 60  0000 C CNN
 F 1 "MCP6001" H 6200 4400 60  0000 C CNN
 F 2 "" H 6100 3500 60  0000 C CNN
@@
 $EndComp
 $Comp
-L +5V #PWR?
+L +5V #PWR37
 U 1 1 516CC87F
 P 6450 3150
-F 0 "#PWR?" H 6450 3240 20  0001 C CNN
+F 0 "#PWR37" H 6450 3240 20  0001 C CNN
 F 1 "+5V" H 6450 3240 30  0000 C CNN
 F 2 "" H 6450 3150 60  0000 C CNN
@@
 $EndComp
 $Comp
-L GND #PWR?
+L GND #PWR38
 U 1 1 516CC885
 P 6450 4400
-F 0 "#PWR?" H 6450 4400 30  0001 C CNN
+F 0 "#PWR38" H 6450 4400 30  0001 C CNN
 F 1 "GND" H 6450 4330 30  0001 C CNN
 F 2 "" H 6450 4400 60  0000 C CNN
@@
 Connection ~ 7250 3750
 $Comp
-L C C?
+L C C14
 U 1 1 516E8E76
 P 4950 2500
-F 0 "C?" H 4950 2600 40  0000 L CNN
+F 0 "C14" H 4950 2600 40  0000 L CNN
 F 1 "100nF" H 4956 2415 40  0000 L CNN
 F 2 "~" H 4988 2350 30  0000 C CNN
@@
 $EndComp
 $Comp
-L +5V #PWR?
+L +5V #PWR33
 U 1 1 516E8E83
 P 4950 2250
-F 0 "#PWR?" H 4950 2340 20  0001 C CNN
+F 0 "#PWR33" H 4950 2340 20  0001 C CNN
 F 1 "+5V" H 4950 2340 30  0000 C CNN
 F 2 "" H 4950 2250 60  0000 C CNN
@@
 $EndComp
 $Comp
-L GND #PWR?
+L GND #PWR34
 U 1 1 516E8E8F
 P 4950 2750
-F 0 "#PWR?" H 4950 2750 30  0001 C CNN
+F 0 "#PWR34" H 4950 2750 30  0001 C CNN
 F 1 "GND" H 4950 2680 30  0001 C CNN
 F 2 "" H 4950 2750 60  0000 C CNN
@@
 	4950 2700 4950 2750
 $Comp
-L C C?
+L C C15
 U 1 1 516E8ED2
 P 6350 2500
-F 0 "C?" H 6350 2600 40  0000 L CNN
+F 0 "C15" H 6350 2600 40  0000 L CNN
 F 1 "100nF" H 6356 2415 40  0000 L CNN
 F 2 "~" H 6388 2350 30  0000 C CNN
@@
 $EndComp
 $Comp
-L +5V #PWR?
+L +5V #PWR35
 U 1 1 516E8ED8
 P 6350 2250
-F 0 "#PWR?" H 6350 2340 20  0001 C CNN
+F 0 "#PWR35" H 6350 2340 20  0001 C CNN
 F 1 "+5V" H 6350 2340 30  0000 C CNN
 F 2 "" H 6350 2250 60  0000 C CNN
@@
 $EndComp
 $Comp
-L GND #PWR?
+L GND #PWR36
 U 1 1 516E8EDE
 P 6350 2750
-F 0 "#PWR?" H 6350 2750 30  0001 C CNN
+F 0 "#PWR36" H 6350 2750 30  0001 C CNN
 F 1 "GND" H 6350 2680 30  0001 C CNN
 F 2 "" H 6350 2750 60  0000 C CNN

Commit message: ran an ERC and touched up a couple small issues
Parts:
- renumbered R45 to R49, R46 to R50, R47 to R51
Changed lines of the file:
@@
-EESchema Schematic File Version 2  date 4/18/2013 12:55:47 AM
+EESchema Schematic File Version 2  date 4/18/2013 1:12:38 AM
 LIBS:power
 LIBS:device
@@
 $Descr A4 11693 8268
 encoding utf-8
-Sheet 7 10
+Sheet 6 10
 Title ""
 Date "18 apr 2013"
@@
 $EndComp
 $Comp
-L R R45
+L R R49
 U 1 1 516CAFEF
 P 2450 2550
-F 0 "R45" V 2530 2550 40  0000 C CNN
+F 0 "R49" V 2530 2550 40  0000 C CNN
 F 1 "R" V 2457 2551 40  0000 C CNN
 F 2 "~" V 2380 2550 30  0000 C CNN
@@
 	2700 3350 2700 2550
 $Comp
-L +5V #PWR31
+L +5V #PWR039
 U 1 1 516CB005
 P 4150 2700
-F 0 "#PWR31" H 4150 2790 20  0001 C CNN
+F 0 "#PWR039" H 4150 2790 20  0001 C CNN
 F 1 "+5V" H 4150 2790 30  0000 C CNN
 F 2 "" H 4150 2700 60  0000 C CNN
@@
 	4150 2700 4150 2850
 $Comp
-L GND #PWR32
+L GND #PWR040
 U 1 1 516CB018
 P 4400 3050
-F 0 "#PWR32" H 4400 3050 30  0001 C CNN
+F 0 "#PWR040" H 4400 3050 30  0001 C CNN
 F 1 "GND" H 4400 2980 30  0001 C CNN
 F 2 "" H 4400 3050 60  0000 C CNN
@@
 	4300 2900 4300 3000
 $Comp
-L R R46
+L R R50
 U 1 1 516CB283
 P 7250 4150
-F 0 "R46" V 7330 4150 40  0000 C CNN
+F 0 "R50" V 7330 4150 40  0000 C CNN
 F 1 "680" V 7257 4151 40  0000 C CNN
 F 2 "~" V 7180 4150 30  0000 C CNN
@@
 $EndComp
 $Comp
-L R R47
+L R R51
 U 1 1 516CB291
 P 7250 4750
-F 0 "R47" V 7330 4750 40  0000 C CNN
+F 0 "R51" V 7330 4750 40  0000 C CNN
 F 1 "1K" V 7257 4751 40  0000 C CNN
 F 2 "~" V 7180 4750 30  0000 C CNN
@@
 SNS_OUT
 $Comp
-L GND #PWR39
+L GND #PWR041
 U 1 1 516CB2F2
 P 7250 5100
-F 0 "#PWR39" H 7250 5100 30  0001 C CNN
+F 0 "#PWR041" H 7250 5100 30  0001 C CNN
 F 1 "GND" H 7250 5030 30  0001 C CNN
 F 2 "" H 7250 5100 60  0000 C CNN
@@
 $EndComp
 $Comp
-L +5V #PWR37
+L +5V #PWR042
 U 1 1 516CC87F
 P 6450 3150
-F 0 "#PWR37" H 6450 3240 20  0001 C CNN
+F 0 "#PWR042" H 6450 3240 20  0001 C CNN
 F 1 "+5V" H 6450 3240 30  0000 C CNN
 F 2 "" H 6450 3150 60  0000 C CNN
@@
 $EndComp
 $Comp
-L GND #PWR38
+L GND #PWR043
 U 1 1 516CC885
 P 6450 4400
-F 0 "#PWR38" H 6450 4400 30  0001 C CNN
+F 0 "#PWR043" H 6450 4400 30  0001 C CNN
 F 1 "GND" H 6450 4330 30  0001 C CNN
 F 2 "" H 6450 4400 60  0000 C CNN
@@
 $EndComp
 $Comp
-L +5V #PWR33
+L +5V #PWR044
 U 1 1 516E8E83
 P 4950 2250
-F 0 "#PWR33" H 4950 2340 20  0001 C CNN
+F 0 "#PWR044" H 4950 2340 20  0001 C CNN
 F 1 "+5V" H 4950 2340 30  0000 C CNN
 F 2 "" H 4950 2250 60  0000 C CNN
@@
 $EndComp
 $Comp
-L GND #PWR34
+L GND #PWR045
 U 1 1 516E8E8F
 P 4950 2750
-F 0 "#PWR34" H 4950 2750 30  0001 C CNN
+F 0 "#PWR045" H 4950 2750 30  0001 C CNN
 F 1 "GND" H 4950 2680 30  0001 C CNN
 F 2 "" H 4950 2750 60  0000 C CNN
@@
 $EndComp
 $Comp
-L +5V #PWR35
+L +5V #PWR046
 U 1 1 516E8ED8
 P 6350 2250
-F 0 "#PWR35" H 6350 2340 20  0001 C CNN
+F 0 "#PWR046" H 6350 2340 20  0001 C CNN
 F 1 "+5V" H 6350 2340 30  0000 C CNN
 F 2 "" H 6350 2250 60  0000 C CNN
@@
 $EndComp
 $Comp
-L GND #PWR36
+L GND #PWR047
 U 1 1 516E8EDE
 P 6350 2750
-F 0 "#PWR36" H 6350 2750 30  0001 C CNN
+F 0 "#PWR047" H 6350 2750 30  0001 C CNN
 F 1 "GND" H 6350 2680 30  0001 C CNN
 F 2 "" H 6350 2750 60  0000 C CNN
