File: power-supply.sch (KiCad schematic (older format))
At the start: 26 parts, among them U2 RT7247AHGSP, U3 LM1117

Commit message: ran an ERC and touched up a couple small issues
Parts:
- gave numbers to parts that had none: 4
- renumbered 12V to 12V1, 3V3 to 3V1, 5V to 5V1, PWR to PWR1, R41 to R45, R42 to R46, R43 to R47, R44 to R48
Connections:
- net GND: now also U2.9 (GND_PAD)
Changed lines of the file:
@@
-EESchema Schematic File Version 2  date 4/18/2013 12:55:47 AM
+EESchema Schematic File Version 2  date 4/18/2013 1:12:38 AM
 LIBS:power
 LIBS:device
@@
 $EndComp
 $Comp
-L GND #PWR22
+L GND #PWR021
 U 1 1 516B7ADE
 P 3000 4100
-F 0 "#PWR22" H 3000 4100 30  0001 C CNN
+F 0 "#PWR021" H 3000 4100 30  0001 C CNN
 F 1 "GND" H 3000 4030 30  0001 C CNN
 F 2 "" H 3000 4100 60  0000 C CNN
@@
 $EndComp
 $Comp
-L R R43
+L R R47
 U 1 1 516B7B34
 P 6650 3650
-F 0 "R43" V 6730 3650 40  0000 C CNN
+F 0 "R47" V 6730 3650 40  0000 C CNN
 F 1 "62k" V 6657 3651 40  0000 C CNN
 F 2 "~" V 6580 3650 30  0000 C CNN
@@
 $EndComp
 $Comp
-L R R44
+L R R48
 U 1 1 516B7B41
 P 6650 4350
-F 0 "R44" V 6730 4350 40  0000 C CNN
+F 0 "R48" V 6730 4350 40  0000 C CNN
 F 1 "11.8k" V 6657 4351 40  0000 C CNN
 F 2 "~" V 6580 4350 30  0000 C CNN
@@
 $EndComp
 $Comp
-L R R42
+L R R46
 U 1 1 516B7B67
 P 5300 4300
-F 0 "R42" V 5380 4300 40  0000 C CNN
+F 0 "R46" V 5380 4300 40  0000 C CNN
 F 1 "20k" V 5307 4301 40  0000 C CNN
 F 2 "~" V 5230 4300 30  0000 C CNN
@@
 $EndComp
 $Comp
-L GND #PWR24
+L GND #PWR022
 U 1 1 516B7CE2
 P 5400 4750
-F 0 "#PWR24" H 5400 4750 30  0001 C CNN
+F 0 "#PWR022" H 5400 4750 30  0001 C CNN
 F 1 "GND" H 5400 4680 30  0001 C CNN
 F 2 "" H 5400 4750 60  0000 C CNN
@@
 $EndComp
 $Comp
-L GND #PWR25
+L GND #PWR023
 U 1 1 516B7CE8
 P 6650 4750
-F 0 "#PWR25" H 6650 4750 30  0001 C CNN
+F 0 "#PWR023" H 6650 4750 30  0001 C CNN
 F 1 "GND" H 6650 4680 30  0001 C CNN
 F 2 "" H 6650 4750 60  0000 C CNN
@@
 $EndComp
 $Comp
-L GND #PWR26
+L GND #PWR024
 U 1 1 516B7DE8
 P 7000 3850
-F 0 "#PWR26" H 7000 3850 30  0001 C CNN
+F 0 "#PWR024" H 7000 3850 30  0001 C CNN
 F 1 "GND" H 7000 3780 30  0001 C CNN
 F 2 "" H 7000 3850 60  0000 C CNN
@@
 $EndComp
 $Comp
-L +5V #PWR27
+L +5V #PWR025
 U 1 1 516B7E14
 P 7150 3200
-F 0 "#PWR27" H 7150 3290 20  0001 C CNN
+F 0 "#PWR025" H 7150 3290 20  0001 C CNN
 F 1 "+5V" H 7150 3290 30  0000 C CNN
 F 2 "" H 7150 3200 60  0000 C CNN
@@
 $EndComp
 $Comp
-L GND #PWR28
+L GND #PWR026
 U 1 1 516B7EDB
 P 7850 2950
-F 0 "#PWR28" H 7850 2950 30  0001 C CNN
+F 0 "#PWR026" H 7850 2950 30  0001 C CNN
 F 1 "GND" H 7850 2880 30  0001 C CNN
 F 2 "" H 7850 2950 60  0000 C CNN
@@
 $EndComp
 $Comp
-L +3.3V #PWR29
+L +3.3V #PWR027
 U 1 1 516B7F0C
 P 8150 3200
-F 0 "#PWR29" H 8150 3160 30  0001 C CNN
+F 0 "#PWR027" H 8150 3160 30  0001 C CNN
 F 1 "+3.3V" H 8150 3310 30  0000 C CNN
 F 2 "" H 8150 3200 60  0000 C CNN
@@
 $EndComp
 $Comp
-L GND #PWR30
+L GND #PWR028
 U 1 1 516B7F4A
 P 8150 3850
-F 0 "#PWR30" H 8150 3850 30  0001 C CNN
+F 0 "#PWR028" H 8150 3850 30  0001 C CNN
 F 1 "GND" H 8150 3780 30  0001 C CNN
 F 2 "" H 8150 3850 60  0000 C CNN
@@
 $EndComp
 $Comp
-L R R41
+L R R45
 U 1 1 516B81BC
 P 3550 3350
-F 0 "R41" V 3630 3350 40  0000 C CNN
+F 0 "R45" V 3630 3350 40  0000 C CNN
 F 1 "100k" V 3557 3351 40  0000 C CNN
 F 2 "~" V 3480 3350 30  0000 C CNN
@@
 $EndComp
 $Comp
-L +5V #PWR23
+L +5V #PWR029
 U 1 1 516B87A2
 P 5300 2650
-F 0 "#PWR23" H 5300 2740 20  0001 C CNN
+F 0 "#PWR029" H 5300 2740 20  0001 C CNN
 F 1 "+5V" H 5300 2740 30  0000 C CNN
 F 2 "" H 5300 2650 60  0000 C CNN
@@
 $EndComp
 $Comp
-L +12V #PWR21
+L +12V #PWR030
 U 1 1 516D7A31
 P 2800 3100
-F 0 "#PWR21" H 2800 3050 20  0001 C CNN
+F 0 "#PWR030" H 2800 3050 20  0001 C CNN
 F 1 "+12V" H 2800 3200 30  0000 C CNN
 F 2 "" H 2800 3100 60  0000 C CNN
@@
 $EndComp
 Wire Wire Line
-	3000 3750 3000 3950
-Wire Wire Line
-	3000 3950 3000 4100
-Wire Wire Line
-	3000 3350 3000 3150
+	3000 3750 3000 4100
+Wire Wire Line
+	3000 3150 3000 3350
 Wire Wire Line
 	3900 3550 3900 3450
@@
 	3000 3950 3250 3950
 Wire Wire Line
-	3250 4000 3700 4000
-Wire Wire Line
-	3700 4000 3900 4000
-Wire Wire Line
-	3900 4000 4050 4000
+	3250 4000 4050 4000
 Wire Wire Line
 	3900 4000 3900 3950
@@
 	5300 3600 5300 3550
 Wire Wire Line
-	5250 3550 5300 3550
-Wire Wire Line
-	5300 3550 5550 3550
+	5250 3550 5550 3550
 Wire Wire Line
 	5550 3550 5550 3600
@@
 	5550 4600 5550 4000
 Wire Wire Line
-	5300 4600 5400 4600
-Wire Wire Line
-	5400 4600 5550 4600
+	5300 4600 5550 4600
 Wire Wire Line
 	5300 4600 5300 4550
@@
 	5300 4050 5300 4000
 Wire Wire Line
-	5250 3300 5800 3300
-Wire Wire Line
-	5800 3300 5950 3300
+	5250 3300 5950 3300
 Wire Wire Line
 	5250 3450 5800 3450
@@
 	5800 4000 6650 4000
 Wire Wire Line
-	6650 3900 6650 4000
-Wire Wire Line
-	6650 4000 6650 4100
+	6650 3900 6650 4100
 Connection ~ 6650 4000
 Wire Wire Line
 	6650 3400 6650 3300
 Wire Wire Line
-	6550 3300 6650 3300
-Wire Wire Line
-	6650 3300 7000 3300
-Wire Wire Line
-	7000 3300 7150 3300
-Wire Wire Line
-	7150 3300 7250 3300
+	6550 3300 7250 3300
 Wire Wire Line
 	5800 3450 5800 4000
 Wire Wire Line
-	5250 3150 5300 3150
-Wire Wire Line
-	5300 3150 5350 3150
+	5250 3150 5350 3150
 Wire Wire Line
 	5800 3150 5750 3150
@@
 	8050 3300 8150 3300
 Wire Wire Line
-	8150 3200 8150 3300
-Wire Wire Line
-	8150 3300 8150 3350
+	8150 3200 8150 3350
 Wire Wire Line
 	8150 3850 8150 3750
@@
 	3300 3350 3200 3350
 Wire Wire Line
-	3200 3350 3200 3150
+	3200 3150 3200 3350
 Connection ~ 3200 3150
 Wire Wire Line
-	3800 3350 3850 3350
-Wire Wire Line
-	3850 3350 4050 3350
+	3800 3350 4050 3350
 Wire Wire Line
 	5300 3100 5300 3150
@@
 	3700 3550 3700 3450
 Wire Wire Line
-	3700 3450 3850 3450
-Wire Wire Line
-	3850 3450 3850 3350
-Wire Wire Line
-	3850 3350 3850 2950
+	3850 3450 3700 3450
+Wire Wire Line
+	3850 2950 3850 3450
 Connection ~ 3850 3350
 Wire Wire Line
@@
 	2650 2800 2750 2800
 Wire Wire Line
-	2450 3150 2800 3150
-Wire Wire Line
-	2800 3150 3000 3150
-Wire Wire Line
-	3000 3150 3200 3150
-Wire Wire Line
-	3200 3150 4050 3150
+	2450 3150 4050 3150
 Wire Wire Line
 	1950 3150 1400 3150
@@
 Connection ~ 2800 3150
 $Comp
-L R R?
+L R R41
 U 1 1 51709AD7
 P 2400 1150
-F 0 "R?" V 2480 1150 40  0000 C CNN
+F 0 "R41" V 2480 1150 40  0000 C CNN
 F 1 "R" V 2407 1151 40  0000 C CNN
 F 2 "~" V 2330 1150 30  0000 C CNN
@@
 $EndComp
 $Comp
-L LED PWR
+L LED PWR1
 U 1 1 51709AE6
 P 2400 1650
-F 0 "PWR" H 2400 1750 50  0000 C CNN
+F 0 "PWR1" H 2400 1750 50  0000 C CNN
 F 1 "LED" H 2400 1550 50  0000 C CNN
 F 2 "~" H 2400 1650 60  0000 C CNN
@@
 $EndComp
 $Comp
-L GND #PWR?
+L GND #PWR031
 U 1 1 51709AF5
 P 2400 1950
-F 0 "#PWR?" H 2400 1950 30  0001 C CNN
+F 0 "#PWR031" H 2400 1950 30  0001 C CNN
 F 1 "GND" H 2400 1880 30  0001 C CNN
 F 2 "" H 2400 1950 60  0000 C CNN
@@
 	2400 750  2400 900
 $Comp
-L R R?
+L R R42
 U 1 1 51709C26
 P 2750 1150
-F 0 "R?" V 2830 1150 40  0000 C CNN
+F 0 "R42" V 2830 1150 40  0000 C CNN
 F 1 "R" V 2757 1151 40  0000 C CNN
 F 2 "~" V 2680 1150 30  0000 C CNN
@@
 $EndComp
 $Comp
-L LED 12V
+L LED 12V1
 U 1 1 51709C2C
 P 2750 1650
-F 0 "12V" H 2750 1750 50  0000 C CNN
+F 0 "12V1" H 2750 1750 50  0000 C CNN
 F 1 "LED" H 2750 1550 50  0000 C CNN
 F 2 "~" H 2750 1650 60  0000 C CNN
@@
 $EndComp
 $Comp
-L GND #PWR?
+L GND #PWR032
 U 1 1 51709C32
 P 2750 1950
-F 0 "#PWR?" H 2750 1950 30  0001 C CNN
+F 0 "#PWR032" H 2750 1950 30  0001 C CNN
 F 1 "GND" H 2750 1880 30  0001 C CNN
 F 2 "" H 2750 1950 60  0000 C CNN
@@
 	2750 1450 2750 1400
 $Comp
-L +12V #PWR?
+L +12V #PWR033
 U 1 1 51709C3A
 P 2750 850
-F 0 "#PWR?" H 2750 800 20  0001 C CNN
+F 0 "#PWR033" H 2750 800 20  0001 C CNN
 F 1 "+12V" H 2750 950 30  0000 C CNN
 F 2 "" H 2750 850 60  0000 C CNN
@@
 	2750 900  2750 850
 $Comp
-L R R?
+L R R43
 U 1 1 51709C41
 P 3050 1150
-F 0 "R?" V 3130 1150 40  0000 C CNN
+F 0 "R43" V 3130 1150 40  0000 C CNN
 F 1 "R" V 3057 1151 40  0000 C CNN
 F 2 "~" V 2980 1150 30  0000 C CNN
@@
 $EndComp
 $Comp
-L LED 5V
+L LED 5V1
 U 1 1 51709C47
 P 3050 1650
-F 0 "5V" H 3050 1750 50  0000 C CNN
+F 0 "5V1" H 3050 1750 50  0000 C CNN
 F 1 "LED" H 3050 1550 50  0000 C CNN
 F 2 "~" H 3050 1650 60  0000 C CNN
@@
 $EndComp
 $Comp
-L GND #PWR?
+L GND #PWR034
 U 1 1 51709C4D
 P 3050 1950
-F 0 "#PWR?" H 3050 1950 30  0001 C CNN
+F 0 "#PWR034" H 3050 1950 30  0001 C CNN
 F 1 "GND" H 3050 1880 30  0001 C CNN
 F 2 "" H 3050 1950 60  0000 C CNN
@@
 	3050 900  3050 850
 $Comp
-L R R?
+L R R44
 U 1 1 51709C5C
 P 3350 1150
-F 0 "R?" V 3430 1150 40  0000 C CNN
+F 0 "R44" V 3430 1150 40  0000 C CNN
 F 1 "R" V 3357 1151 40  0000 C CNN
 F 2 "~" V 3280 1150 30  0000 C CNN
@@
 $EndComp
 $Comp
-L LED 3V3
+L LED 3V1
 U 1 1 51709C62
 P 3350 1650
-F 0 "3V3" H 3350 1750 50  0000 C CNN
+F 0 "3V1" H 3350 1750 50  0000 C CNN
 F 1 "LED" H 3350 1550 50  0000 C CNN
 F 2 "~" H 3350 1650 60  0000 C CNN
@@
 $EndComp
 $Comp
-L GND #PWR?
+L GND #PWR035
 U 1 1 51709C68
 P 3350 1950
-F 0 "#PWR?" H 3350 1950 30  0001 C CNN
+F 0 "#PWR035" H 3350 1950 30  0001 C CNN
 F 1 "GND" H 3350 1880 30  0001 C CNN
 F 2 "" H 3350 1950 60  0000 C CNN
@@
 	3350 900  3350 850
 $Comp
-L +5V #PWR?
+L +5V #PWR036
 U 1 1 51709C77
 P 3050 850
-F 0 "#PWR?" H 3050 940 20  0001 C CNN
+F 0 "#PWR036" H 3050 940 20  0001 C CNN
 F 1 "+5V" H 3050 940 30  0000 C CNN
 F 2 "" H 3050 850 60  0000 C CNN
@@
 $EndComp
 $Comp
-L +3.3V #PWR?
+L +3.3V #PWR037
 U 1 1 51709C8E
 P 3350 850
-F 0 "#PWR?" H 3350 810 30  0001 C CNN
+F 0 "#PWR037" H 3350 810 30  0001 C CNN
 F 1 "+3.3V" H 3350 960 30  0000 C CNN
 F 2 "" H 3350 850 60  0000 C CNN
@@
 Wire Wire Line
 	2300 750  2400 750
+$Comp
+L GND #PWR038
+U 1 1 5170A047
+P 4650 4050
+F 0 "#PWR038" H 4650 4050 30  0001 C CNN
+F 1 "GND" H 4650 3980 30  0001 C CNN
+F 2 "" H 4650 4050 60  0000 C CNN
+F 3 "" H 4650 4050 60  0000 C CNN
+	1    4650 4050
+	1    0    0    -1
+$EndComp
+Wire Wire Line
+	4650 4050 4650 4000
 $EndSCHEMATC

Commit message: added some more info to the different components, changed the pinout for zeeners, and am hating ki-cad for schematic to pads.
Changed lines of the file:
@@
-EESchema Schematic File Version 2  date 4/18/2013 1:12:38 AM
+EESchema Schematic File Version 2  date 4/19/2013 12:46:09 AM
 LIBS:power
 LIBS:device
@@
 Sheet 5 10
 Title ""
-Date "18 apr 2013"
+Date "19 apr 2013"
 Rev ""
 Comp ""
@@
 F 1 "15uH" V 6350 3300 40  0000 C CNN
 F 2 "~" H 6250 3300 60  0000 C CNN
-F 3 "~" H 6250 3300 60  0000 C CNN
+F 3 "445-3579-1-ND" H 6250 3300 60  0000 C CNN
 	1    6250 3300
 	0    -1   -1   0
@@
 	3300 3350 3200 3350
 Wire Wire Line
-	3200 3150 3200 3350
+	3200 3350 3200 3150
 Connection ~ 3200 3150
 Wire Wire Line
@@
 	3700 3550 3700 3450
 Wire Wire Line
-	3850 3450 3700 3450
-Wire Wire Line
-	3850 2950 3850 3450
+	3700 3450 3850 3450
+Wire Wire Line
+	3850 3450 3850 2950
 Connection ~ 3850 3350
 Wire Wire Line
