File: rgb-led-output.sch (KiCad schematic (older format))
At the start: 9 parts, among them K1 CONN_3, Q32 BSS138, U8 LM7805CT

Commit message: Fixing reversed 5V regulator and adding polarized header for WS2812B strip output.
Parts:
- K1: footprint Socket_Strips:Socket_Strip_Straight_1x03 -> Sockets_MOLEX_KK-System:Socket_MOLEX-KK-RM2-54mm_Lock_3pin_straight
Changed lines of the file:
@@
 F 0 "K1" V 5550 3700 50  0000 C CNN
 F 1 "CONN_3" V 5650 3700 40  0000 C CNN
-F 2 "Socket_Strips:Socket_Strip_Straight_1x03" H 5600 3700 60  0001 C BNN
+F 2 "Sockets_MOLEX_KK-System:Socket_MOLEX-KK-RM2-54mm_Lock_3pin_straight" H 5600 3700 60  0001 C BNN
 F 3 "" H 5600 3700 60  0000 C CNN
 	1    5600 3700
