File: 2.x/accelerometer.sch (KiCad schematic (older format))
At the start: 5 parts, among them U9 MMA8653FC

Commit message: Committing latest files. This includes the KiCAD 4.0.0rc1 migration as well as the updates to Base Board 2.1.
Parts:
- C23, C24, C25, C26: symbol C -> C-RESCUE-base-module-hardware-v2
Changed lines of the file:
@@
 EESchema Schematic File Version 2
+LIBS:base-module-hardware-v2-rescue
 LIBS:power
 LIBS:device
@@
 LIBS:memory
 LIBS:xilinx
-LIBS:special
 LIBS:microcontrollers
 LIBS:dsp
@@
 Connection ~ 5850 3200
 $Comp
-L GND #PWR059
+L GND-RESCUE-base-module-hardware-v2 #PWR061
 U 1 1 5507A530
 P 5850 4800
-F 0 "#PWR059" H 5850 4800 30  0001 C CNN
+F 0 "#PWR061" H 5850 4800 30  0001 C CNN
 F 1 "GND" H 5850 4730 30  0001 C CNN
 F 2 "" H 5850 4800 60  0000 C CNN
@@
 	5950 4700 5950 4600
 $Comp
-L C C23
+L C-RESCUE-base-module-hardware-v2 C23
 U 1 1 5507C820
 P 7000 4000
@@
 $EndComp
 $Comp
-L C C24
+L C-RESCUE-base-module-hardware-v2 C24
 U 1 1 5507C82B
 P 7300 4000
@@
 $EndComp
 $Comp
-L C C25
+L C-RESCUE-base-module-hardware-v2 C25
 U 1 1 5507C85C
 P 7600 4000
@@
 Connection ~ 7300 3200
 $Comp
-L C C26
+L C-RESCUE-base-module-hardware-v2 C26
 U 1 1 5507C903
 P 6150 4900
@@
 $EndComp
 $Comp
-L GND #PWR060
+L GND-RESCUE-base-module-hardware-v2 #PWR062
 U 1 1 5507C932
 P 6150 5200
-F 0 "#PWR060" H 6150 5200 30  0001 C CNN
+F 0 "#PWR062" H 6150 5200 30  0001 C CNN
 F 1 "GND" H 6150 5130 30  0001 C CNN
 F 2 "" H 6150 5200 60  0000 C CNN
@@
 	6150 4700 6150 4600
 $Comp
-L GND #PWR061
+L GND-RESCUE-base-module-hardware-v2 #PWR063
 U 1 1 5507C983
 P 7300 4400
-F 0 "#PWR061" H 7300 4400 30  0001 C CNN
+F 0 "#PWR063" H 7300 4400 30  0001 C CNN
 F 1 "GND" H 7300 4330 30  0001 C CNN
 F 2 "" H 7300 4400 60  0000 C CNN
