File: 2.x/control-logic.sch (KiCad schematic (older format))
At the start: 34 parts, among them U2 STM32F072R, U3 MCP2562, X1 8.000 MHz

Commit message: Committing latest files. This includes the KiCAD 4.0.0rc1 migration as well as the updates to Base Board 2.1.
Parts:
- C10, C11, C12, C4, C5, C6, C7, C8, C9: symbol C -> C-RESCUE-base-module-hardware-v2
- R101, R102, R103, R104, R105, R106, R107, R108, R109, R110, R111, R112, R113, R114: symbol R -> R-RESCUE-base-module-hardware-v2
Connections:
- net HEARTBEAT: now also HB1.2 (A); no longer HB1.1 (K)
- net POWER_GOOD: now also PG1.2 (A); no longer PG1.1 (K)
- net at R104.1: now also PG1.1 (K); no longer PG1.2 (A)
- net at R103.1: now also HB1.1 (K); no longer HB1.2 (A)
Changed lines of the file:
@@
 EESchema Schematic File Version 2
+LIBS:base-module-hardware-v2-rescue
 LIBS:power
 LIBS:device
@@
 LIBS:memory
 LIBS:xilinx
-LIBS:special
 LIBS:microcontrollers
 LIBS:dsp
@@
 $EndComp
 $Comp
-L R R114
+L R-RESCUE-base-module-hardware-v2 R114
 U 1 1 5325B4BA
 P 9650 6200
@@
 $EndComp
 $Comp
-L R R113
+L R-RESCUE-base-module-hardware-v2 R113
 U 1 1 5325B4C9
 P 9450 6200
@@
 $EndComp
 $Comp
-L R R112
+L R-RESCUE-base-module-hardware-v2 R112
 U 1 1 5325B4D8
 P 9250 6200
@@
 $EndComp
 $Comp
-L R R111
+L R-RESCUE-base-module-hardware-v2 R111
 U 1 1 5325B4E7
 P 9050 6200
@@
 $EndComp
 $Comp
-L R R110
+L R-RESCUE-base-module-hardware-v2 R110
 U 1 1 5325B4F6
 P 8850 6200
@@
 $EndComp
 $Comp
-L R R109
+L R-RESCUE-base-module-hardware-v2 R109
 U 1 1 5325B505
 P 8650 6200
@@
 $EndComp
 $Comp
-L R R108
+L R-RESCUE-base-module-hardware-v2 R108
 U 1 1 5325B514
 P 8450 6200
@@
 $EndComp
 $Comp
-L R R107
+L R-RESCUE-base-module-hardware-v2 R107
 U 1 1 5325B523
 P 8250 6200
@@
 $EndComp
 $Comp
-L GND #PWR027
+L GND-RESCUE-base-module-hardware-v2 #PWR027
 U 1 1 5325BA22
 P 9050 6650
@@
 VSOL_PRECHARGE_PWM
 $Comp
-L GND #PWR028
+L GND-RESCUE-base-module-hardware-v2 #PWR028
 U 1 1 53262BD9
 P 3050 5600
@@
 $EndComp
 $Comp
-L C C5
+L C-RESCUE-base-module-hardware-v2 C5
 U 1 1 53264A23
 P 1500 2000
@@
 $EndComp
 $Comp
-L C C4
+L C-RESCUE-base-module-hardware-v2 C4
 U 1 1 53264A32
 P 1500 1400
@@
 $EndComp
 $Comp
-L GND #PWR029
+L GND-RESCUE-base-module-hardware-v2 #PWR029
 U 1 1 53264B7B
 P 1200 2100
@@
 $EndComp
 $Comp
-L LED PG1
-U 1 1 53267B24
-P 10100 1250
-F 0 "PG1" H 10100 1350 50  0000 C CNN
-F 1 "LED" H 10100 1150 50  0000 C CNN
-F 2 "LEDs:LED-0603" H 10100 1250 60  0001 C CNN
-F 3 "~" H 10100 1250 60  0000 C CNN
-	1    10100 1250
-	0    1    1    0
-$EndComp
-$Comp
-L LED HB1
-U 1 1 53267B33
-P 9800 1250
-F 0 "HB1" H 9800 1350 50  0000 C CNN
-F 1 "LED" H 9800 1150 50  0000 C CNN
-F 2 "LEDs:LED-0603" H 9800 1250 60  0001 C CNN
-F 3 "~" H 9800 1250 60  0000 C CNN
-	1    9800 1250
-	0    1    1    0
-$EndComp
-$Comp
-L R R102
+L R-RESCUE-base-module-hardware-v2 R102
 U 1 1 53267B42
 P 8500 1100
@@
 $EndComp
 $Comp
-L R R101
+L R-RESCUE-base-module-hardware-v2 R101
 U 1 1 53267B51
 P 8050 1100
@@
 $EndComp
 $Comp
-L R R104
+L R-RESCUE-base-module-hardware-v2 R104
 U 1 1 53267B60
 P 10100 1800
@@
 $EndComp
 $Comp
-L R R103
+L R-RESCUE-base-module-hardware-v2 R103
 U 1 1 53267B6F
 P 9800 1800
@@
 $EndComp
 $Comp
-L C C6
+L C-RESCUE-base-module-hardware-v2 C6
 U 1 1 53267B9C
 P 6350 6150
@@
 $EndComp
 $Comp
-L C C7
+L C-RESCUE-base-module-hardware-v2 C7
 U 1 1 53267BAB
 P 6600 6150
@@
 $EndComp
 $Comp
-L C C8
+L C-RESCUE-base-module-hardware-v2 C8
 U 1 1 53267BBA
 P 6850 6150
@@
 $EndComp
 $Comp
-L C C9
+L C-RESCUE-base-module-hardware-v2 C9
 U 1 1 53267BC9
 P 7100 6150
@@
 $EndComp
 $Comp
-L C C10
+L C-RESCUE-base-module-hardware-v2 C10
 U 1 1 53267BD8
 P 7350 6150
@@
 $EndComp
 $Comp
-L GND #PWR030
+L GND-RESCUE-base-module-hardware-v2 #PWR030
 U 1 1 53268402
 P 6350 6550
@@
 LOCAL_3V3
 $Comp
-L GND #PWR031
+L GND-RESCUE-base-module-hardware-v2 #PWR031
 U 1 1 53268FE5
 P 8050 2250
@@
 $EndComp
 $Comp
-L GND #PWR032
+L GND-RESCUE-base-module-hardware-v2 #PWR032
 U 1 1 532697A4
 P 9950 2250
@@
 POWER_GOOD
 $Comp
-L GND #PWR033
+L GND-RESCUE-base-module-hardware-v2 #PWR033
 U 1 1 5326A151
 P 7850 3100
@@
 TXD
 $Comp
-L GND #PWR034
+L GND-RESCUE-base-module-hardware-v2 #PWR034
 U 1 1 5326B790
 P 10000 3100
@@
 SDA
 $Comp
-L GND #PWR035
+L GND-RESCUE-base-module-hardware-v2 #PWR035
 U 1 1 533CA56F
 P 9100 4150
@@
 $EndComp
 $Comp
-L R R106
+L R-RESCUE-base-module-hardware-v2 R106
 U 1 1 533CAC4E
 P 8950 3650
@@
 $EndComp
 $Comp
-L R R105
+L R-RESCUE-base-module-hardware-v2 R105
 U 1 1 533CAE0E
 P 8750 3650
@@
 $EndComp
 $Comp
-L GND #PWR036
+L GND-RESCUE-base-module-hardware-v2 #PWR036
 U 1 1 54EC01AF
 P 2200 7650
@@
 LOCAL_5V
 $Comp
-L C C11
+L C-RESCUE-base-module-hardware-v2 C11
 U 1 1 54EC1BB5
 P 3750 7250
@@
 $EndComp
 $Comp
-L C C12
+L C-RESCUE-base-module-hardware-v2 C12
 U 1 1 54EC1E37
 P 4050 7250
@@
 $EndComp
 $Comp
-L GND #PWR037
+L GND-RESCUE-base-module-hardware-v2 #PWR037
 U 1 1 54EC1E75
 P 3900 7650
@@
 Wire Wire Line
 	4050 3800 4450 3800
+$Comp
+L LED PG1
+U 1 1 5611DBC4
+P 10100 1250
+F 0 "PG1" H 10100 1350 50  0000 C CNN
+F 1 "LED" H 10100 1150 50  0000 C CNN
+F 2 "LEDs:LED-0603" H 10100 1250 60  0001 C CNN
+F 3 "" H 10100 1250 60  0000 C CNN
+	1    10100 1250
+	0    -1   -1   0
+$EndComp
+$Comp
+L LED HB1
+U 1 1 5611DCCF
+P 9800 1250
+F 0 "HB1" H 9800 1350 50  0000 C CNN
+F 1 "LED" H 9800 1150 50  0000 C CNN
+F 2 "LEDs:LED-0603" H 9800 1250 60  0001 C CNN
+F 3 "" H 9800 1250 60  0000 C CNN
+	1    9800 1250
+	0    -1   -1   0
+$EndComp
 $EndSCHEMATC
